File: hardware/battery-management-system/cell_balancing.kicad_sch (KiCad schematic)
At the start: 48 parts, among them IC1 LT8584EFE#PBF, IC2 LT8584EFE#PBF, IC3 LT8584EFE#PBF, IC4 LT8584EFE#PBF, T1 NA6252-ALD, T2 NA6252-ALD, T3 NA6252-ALD, T4 NA6252-ALD

Commit message: update symbols from library
Parts:
- C40, C47, C54, C61: Mouser Part Number 80-C0603C223K4RAC -> 80-C0603C223K4RAC
- R45, R46, R47, R48: Mouser Part Number (none) -> 652-CR0603FX-4701ELF
Changed lines of the file:
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@@
 			)
 		)
+		(property "Mouser Part Number" "652-CR0603FX-4701ELF"
+			(at 124.46 73.66 0)
+			(effects
+				(font
+					(size 1.27 1.27)
+				)
+				(hide yes)
+			)
+		)
 		(pin "2"
 		)
@@
 			)
 		)
-		(property "Mouser Part Number" " 80-C0603C223K4RAC"
+		(property "Mouser Part Number" "80-C0603C223K4RAC"
 			(at 159.766 19.05 0)
 			(effects
@@
 			)
 		)
-		(property "Mouser Part Number" " 80-C0603C223K4RAC"
+		(property "Mouser Part Number" "80-C0603C223K4RAC"
 			(at 159.766 107.95 0)
 			(effects
@@
 			)
 		)
+		(property "Mouser Part Number" "652-CR0603FX-4701ELF"
+			(at 124.46 162.56 0)
+			(effects
+				(font
+					(size 1.27 1.27)
+				)
+				(hide yes)
+			)
+		)
 		(pin "2"
 		)
@@
 			)
 		)
-		(property "Mouser Part Number" " 80-C0603C223K4RAC"
+		(property "Mouser Part Number" "80-C0603C223K4RAC"
 			(at 159.766 152.4 0)
 			(effects
@@
 			)
 		)
+		(property "Mouser Part Number" "652-CR0603FX-4701ELF"
+			(at 124.46 29.21 0)
+			(effects
+				(font
+					(size 1.27 1.27)
+				)
+				(hide yes)
+			)
+		)
 		(pin "2"
 		)
@@
 			)
 		)
+		(property "Mouser Part Number" "652-CR0603FX-4701ELF"
+			(at 124.46 118.11 0)
+			(effects
+				(font
+					(size 1.27 1.27)
+				)
+				(hide yes)
+			)
+		)
 		(pin "2"
 		)
@@
 			)
 		)
-		(property "Mouser Part Number" " 80-C0603C223K4RAC"
+		(property "Mouser Part Number" "80-C0603C223K4RAC"
 			(at 159.766 63.5 0)
 			(effects

Commit message: update symbols from library
Parts:
- D17, D18, D19, D20: Mouser Part Number (none) -> 621-SBR2065D1-13
Changed lines of the file:
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@@
+			)
+		)
+		(property "Mouser Part Number" "621-SBR2065D1-13"
+			(at 184.404 21.59 0)
+			(effects
+				(font
+					(size 1.27 1.27)
+				)
+				(hide yes)
 			)
 		)
@@
 			)
 		)
+		(property "Mouser Part Number" "621-SBR2065D1-13"
+			(at 184.404 110.49 0)
+			(effects
+				(font
+					(size 1.27 1.27)
+				)
+				(hide yes)
+			)
+		)
 		(pin "2"
 		)
@@
 			)
 		)
+		(property "Mouser Part Number" "621-SBR2065D1-13"
+			(at 184.404 66.04 0)
+			(effects
+				(font
+					(size 1.27 1.27)
+				)
+				(hide yes)
+			)
+		)
 		(pin "2"
 		)
@@
 			(at 184.404 154.94 0)
 			(effects
+				(font
+					(size 1.27 1.27)
+				)
+				(hide yes)
+			)
+		)
+		(property "Mouser Part Number" "621-SBR2065D1-13"
+			(at 184.404 154.94 0)
+			(effects

Commit message: update symbols
Parts:
- C40, C47, C54, C61: Mouser Part Number 80-C0603C223K4RAC -> 80-C0603C223K4R
Changed lines of the file:
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@@
 			)
 		)
-		(property "Mouser Part Number" "80-C0603C223K4RAC"
+		(property "Mouser Part Number" "80-C0603C223K4R"
 			(at 159.766 19.05 0)
 			(effects
@@
 			)
 		)
-		(property "Mouser Part Number" "80-C0603C223K4RAC"
+		(property "Mouser Part Number" "80-C0603C223K4R"
 			(at 159.766 107.95 0)
 			(effects
@@
 			)
 		)
-		(property "Mouser Part Number" "80-C0603C223K4RAC"
+		(property "Mouser Part Number" "80-C0603C223K4R"
 			(at 159.766 152.4 0)
 			(effects
@@
 			)
 		)
-		(property "Mouser Part Number" "80-C0603C223K4RAC"
+		(property "Mouser Part Number" "80-C0603C223K4R"
 			(at 159.766 63.5 0)
 			(effects

Commit message: update symbols and BOM
Parts:
- C46, C53, C60, C67: Mouser Part Number 80-C0603C473K4RAC -> 80-C0603C473K4RACLR
Changed lines of the file:
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@@
 			)
 		)
-		(property "Mouser Part Number" "80-C0603C473K4RAC"
+		(property "Mouser Part Number" "80-C0603C473K4RACLR"
 			(at 89.916 134.62 0)
 			(effects
@@
 			)
 		)
-		(property "Mouser Part Number" "80-C0603C473K4RAC"
+		(property "Mouser Part Number" "80-C0603C473K4RACLR"
 			(at 89.916 179.07 0)
 			(effects
@@
 			)
 		)
-		(property "Mouser Part Number" "80-C0603C473K4RAC"
+		(property "Mouser Part Number" "80-C0603C473K4RACLR"
 			(at 89.916 90.17 0)
 			(effects
@@
 			)
 		)
-		(property "Mouser Part Number" "80-C0603C473K4RAC"
+		(property "Mouser Part Number" "80-C0603C473K4RACLR"
 			(at 89.916 45.72 0)
 			(effects
