File: hardware/battery-management-system/usb.kicad_sch (KiCad schematic)
At the start: 20 parts, among them J5 AMPHENOL_micro_usb_10118194-0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, U6 FT230XS

Commit message: update symbols from library
Parts:
- C16: Mouser Part Number (none) -> 187-CL21A475KBQNNNE
- C19, C20: Mouser Part Number (none) -> 791-0603N470J101CT
- R19, R20, R21, R22: Mouser Part Number (none) -> 652-CR0603FX-1002ELF
Changed lines of the file:
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@@
+			)
+		)
+		(property "Mouser Part Number" "652-CR0603FX-1002ELF"
+			(at 132.08 74.93 0)
+			(effects
+				(font
+					(size 1.27 1.27)
+				)
+				(hide yes)
 			)
 		)
@@
 			)
 		)
+		(property "Mouser Part Number" "187-CL21A475KBQNNNE"
+			(at 89.916 78.74 0)
+			(effects
+				(font
+					(size 1.27 1.27)
+				)
+				(hide yes)
+			)
+		)
 		(pin "1"
 		)
@@
 			)
 		)
+		(property "Mouser Part Number" "652-CR0603FX-1002ELF"
+			(at 144.78 74.93 0)
+			(effects
+				(font
+					(size 1.27 1.27)
+				)
+				(hide yes)
+			)
+		)
 		(pin "1"
 		)
@@
 			)
 		)
+		(property "Mouser Part Number" "652-CR0603FX-1002ELF"
+			(at 157.48 74.93 0)
+			(effects
+				(font
+					(size 1.27 1.27)
+				)
+				(hide yes)
+			)
+		)
 		(pin "1"
 		)
@@
 			)
 		)
+		(property "Mouser Part Number" "652-CR0603FX-1002ELF"
+			(at 170.18 74.93 0)
+			(effects
+				(font
+					(size 1.27 1.27)
+				)
+				(hide yes)
+			)
+		)
 		(pin "1"
 		)
@@
 			)
 		)
+		(property "Mouser Part Number" "791-0603N470J101CT"
+			(at 92.456 110.49 0)
+			(effects
+				(font
+					(size 1.27 1.27)
+				)
+				(hide yes)
+			)
+		)
 		(pin "1"
 		)
@@
 			(at 105.156 110.49 0)
 			(effects
+				(font
+					(size 1.27 1.27)
+				)
+				(hide yes)
+			)
+		)
+		(property "Mouser Part Number" "791-0603N470J101CT"
+			(at 105.156 110.49 0)
+			(effects

Commit message: update symbols from library
Parts:
- D12: Mouser Part Number (none) -> 604-AP1608SGC
- D13: Mouser Part Number (none) -> 604-APH1608SURCK
- FB1: Mouser Part Number (none) -> 81-BLM11P300S
- J5: Mouser Part Number (none) -> 649-10118194-0001LF
- R15, R16: Mouser Part Number (none) -> 603-RC0603FR-0727RL
- R17, R18: Mouser Part Number (none) -> 603-RC0603FR-07120RL
- U6: Mouser Part Number (none) -> 895-FT230XS-R
Changed lines of the file:
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@@
+			)
+		)
+		(property "Mouser Part Number" "895-FT230XS-R"
+			(at 125.73 95.25 0)
+			(effects
+				(font
+					(size 1.27 1.27)
+				)
+				(hide yes)
 			)
 		)
@@
 			)
 		)
+		(property "Mouser Part Number" "604-APH1608SURCK"
+			(at 218.44 76.2 0)
+			(effects
+				(font
+					(size 1.27 1.27)
+				)
+				(hide yes)
+			)
+		)
 		(pin "1"
 		)
@@
 			)
 		)
+		(property "Mouser Part Number" "81-BLM11P300S"
+			(at 85.09 36.83 0)
+			(effects
+				(font
+					(size 1.27 1.27)
+				)
+				(hide yes)
+			)
+		)
 		(pin "1"
 		)
@@
 			)
 		)
+		(property "Mouser Part Number" "603-RC0603FR-07120RL"
+			(at 200.66 64.77 0)
+			(effects
+				(font
+					(size 1.27 1.27)
+				)
+				(hide yes)
+			)
+		)
 		(pin "1"
 		)
@@
 			)
 		)
+		(property "Mouser Part Number" "603-RC0603FR-0727RL"
+			(at 93.98 59.69 0)
+			(effects
+				(font
+					(size 1.27 1.27)
+				)
+				(hide yes)
+			)
+		)
 		(pin "1"
 		)
@@
 			)
 		)
+		(property "Mouser Part Number" "604-AP1608SGC"
+			(at 201.93 76.2 0)
+			(effects
+				(font
+					(size 1.27 1.27)
+				)
+				(hide yes)
+			)
+		)
 		(pin "1"
 		)
@@
 			)
 		)
+		(property "Mouser Part Number" "603-RC0603FR-07120RL"
+			(at 184.15 64.77 0)
+			(effects
+				(font
+					(size 1.27 1.27)
+				)
+				(hide yes)
+			)
+		)
 		(pin "1"
 		)
@@
 			)
 		)
+		(property "Mouser Part Number" "603-RC0603FR-0727RL"
+			(at 93.98 57.15 0)
+			(effects
+				(font
+					(size 1.27 1.27)
+				)
+				(hide yes)
+			)
+		)
 		(pin "1"
 		)
@@
 			(at 125.73 45.72 0)
 			(effects
+				(font
+					(size 1.27 1.27)
+				)
+				(hide yes)
+			)
+		)
+		(property "Mouser Part Number" "649-10118194-0001LF"
+			(at 125.73 45.72 0)
+			(effects

Commit message: update symbols and BOM
Parts:
- D13: Mouser Part Number 604-APH1608SURCK -> 859-LTST-C190KDKT10A
Changed lines of the file:
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@@
 			)
 		)
-		(property "Mouser Part Number" "604-APH1608SURCK"
+		(property "Mouser Part Number" "859-LTST-C190KDKT10A"
 			(at 218.44 76.2 0)
 			(effects
