File: hardware/cell-temperature-sensor/cell-temperature-sensor.kicad_sch (KiCad schematic)
At the start: 12 parts, among them J1 3V3, J2 SCL, J3 SDA, J4 GND, U9 NCT75DR2G

Commit message: add BOM for cell temperature sensor
Parts:
- C25: Mouser Part Number (none) -> 581-KGM15BR71H104KM
- R1, R2, R3, R4, R5, R6: Mouser Part Number (none) -> 603-RT0603FRE13100KL
- U9: Mouser Part Number (none) -> 863-NCT75DR2G
